Commit message: 1

File: twowheelbot/designs/amrurdf.urdf (robot description, URDF)
Before this commit: robot None, 8 links, 7 joints
Joints:
- joint chassis_joint: origin xyz=0 0 0 rpy=0 0 0 -> xyz=0 0 0.045 rpy=0 0 0

File: twowheelbot/designs/gz_ctrl.xacro (robot description, xacro)
@@ -13,5 +13,5 @@
             <!-- output -->
             <odometry_frame>odom</odometry_frame>
-            <robot_base_frame>base_footprint</robot_base_frame>
+            <robot_base_frame>base_link</robot_base_frame>
             <publish_odom>true</publish_odom>
             <publish_odom_tf>true</publish_odom_tf>

File: twowheelbot/designs/lidar.xacro (robot description, xacro)
@@ -30,14 +30,14 @@
   </joint>
   <gazebo reference="lidar_link">
-    <material>Gazebo/Brown</material>
+    <material>Gazebo/Pink</material>
     <sensor name="laser" type="ray">
         <pose>0 0 0 0 0 0</pose>
         <visualize>false</visualize>
-        <update_ray>10</update_ray>
+        <update_rate>10</update_rate>
         <ray>
             <scan>
                 <horizontal>
                     <samples>360</samples>
-                    <resolution>0.5</resolution>
+                    <!-- <resolution>0.5</resolution> -->
                     <min_angle>-3.14</min_angle>
                     <max_angle>3.14</max_angle>
@@ -46,16 +46,16 @@
             <range>
                 <min>0.1</min>
-                <max>8</max>
+                <max>11</max>
                 <!-- <resoluion>0.05</resoluion> -->
             </range>
-            <noise>
+            <!-- <noise>
                 <type>gaussian</type>
                 <mean>0.0</mean>
                 <stddev>0.01</stddev>
-              </noise>
+            </noise> -->
         </ray>
-        <plugin name = "scan" filename = "libgazebo_ros_ray_sensor.so">
+        <plugin name = "laser_controller" filename = "libgazebo_ros_ray_sensor.so">
             <ros>
-                <argument>--ros-args --remap ~/out:=scan</argument>
+                <argument>~/out:=scan</argument>
             </ros>
             <output_type>sensor_msgs/LaserScan</output_type>
