Commit message: twowheelbot final update
Resolved Lidar issues and added diff drive control

File: twowheelbot/designs/amr.urdf.xacro (robot description, xacro)
@@ -2,3 +2,4 @@
 <robot xmlns:xacro="http://www.ros.org/wiki/xacro" name="amr_bot">
     <xacro:include filename = "amrurdf.urdf" />
+    <xacro:include filename = "gz_ctrl.xacro" />
 </robot>

File: twowheelbot/designs/amrurdf.urdf (robot description, URDF)
Before this commit: robot None, 9 links, 8 joints
Joints:
- joint chassis_joint: origin xyz=0 0 0.05 -> xyz=0 0 0
- joint left_wheel_joint: axis 0 0 1 -> 0 0 -1; origin xyz=0 0.234000000000001 0.0304999999999985 rpy=-1.5707963267949 0 0 -> xyz=0 0.234 0.0304999999999985 rpy=-${pi/2} 0 0
- joint lf_caster_joint: origin xyz=0.121999999999999 0.107 -0.0309999999999993 rpy=-1.5707963267949 0 0 -> xyz=0.121999999999999 0.107 -0.028 rpy=-${pi/2} 0 0
- joint lidar_link_joint: origin xyz=-0.0063382 0.0016853 0.193 rpy=0 0 1.5164 -> xyz=-0.0063382 0.0016853 0.225 rpy=0 0 1.5164
- joint lr_caster_joint: origin xyz=-0.154 0.107 -0.0310000000000015 rpy=-1.5707963267949 0 0 -> xyz=-0.154 0.107 -0.028 rpy=-${pi/2} 0 0
- joint rf_caster_joint: origin xyz=0.121999999999999 -0.107 -0.031 rpy=1.5707963267949 0 0 -> xyz=0.121999999999999 -0.107 -0.028 rpy=${pi/2} 0 0
- joint right_wheel_joint: origin xyz=0 -0.234 0.0304999999999984 rpy=1.5707963267949 0 0 -> xyz=0 -0.234 0.0304999999999984 rpy=${pi/2} 0 0
- joint rr_caster_joint: origin xyz=-0.154 -0.107 -0.0310000000000008 rpy=1.5707963267949 0 0 -> xyz=-0.154 -0.107 -0.028 rpy=${pi/2} 0 0

Commit message: Updates
made Lidar.xacro different
Added Imu.xacro, ekf.yaml, caostmap
Many More

File: twowheelbot/designs/amr.urdf.xacro (robot description, xacro)
@@ -3,3 +3,11 @@
     <xacro:include filename = "amrurdf.urdf" />
     <xacro:include filename = "gz_ctrl.xacro" />
+    <xacro:include filename = "lidar.xacro"/>
+    <!-- <xacro:include filename = "imu.xacro"/> -->
+    <!-- <xacro:if value="$(arg use_ros2_control)">
+        <xacro:include filename="ros2_control.xacro" />
+    </xacro:if>
+    <xacro:unless value="$(arg use_ros2_control)">
+        <xacro:include filename="gazebo_control.xacro" />
+    </xacro:unless> -->
 </robot>

File: twowheelbot/designs/amrurdf.urdf (robot description, URDF)
Before this commit: robot None, 9 links, 8 joints
Links:
- removed link lidar_link
Joints:
- removed joint lidar_link_joint
- joint chassis_joint: origin xyz=0 0 0 -> xyz=0 0 0 rpy=0 0 ${pi}

Commit message: SLAM toolbox Integration

File: twowheelbot/designs/amr.urdf.xacro (robot description, xacro)
@@ -2,11 +2,11 @@
 <robot xmlns:xacro="http://www.ros.org/wiki/xacro" name="amr_bot">
     <xacro:include filename = "amrurdf.urdf" />
-    <xacro:include filename = "gz_ctrl.xacro" />
+    <!-- <xacro:include filename = "gz_ctrl.xacro" /> -->
     <xacro:include filename = "lidar.xacro"/>
     <!-- <xacro:include filename = "imu.xacro"/> -->
-    <!-- <xacro:if value="$(arg use_ros2_control)">
+    <!-- <xacro:if value="$(arg use_ros2_control)"> -->
         <xacro:include filename="ros2_control.xacro" />
-    </xacro:if>
-    <xacro:unless value="$(arg use_ros2_control)">
+    <!-- </xacro:if> -->
+    <!-- <xacro:unless value="$(arg use_ros2_control)">
         <xacro:include filename="gazebo_control.xacro" />
     </xacro:unless> -->

File: twowheelbot/designs/amrurdf.urdf (robot description, URDF)
Before this commit: robot None, 8 links, 7 joints
Joints:
- joint chassis_joint: origin xyz=0 0 0 rpy=0 0 ${pi} -> xyz=0 0 0 rpy=0 0 0

File: twowheelbot/designs/gz_ctrl.xacro (robot description, xacro)
@@ -13,5 +13,5 @@
             <!-- output -->
             <odometry_frame>odom</odometry_frame>
-            <robot_base_frame>base_link</robot_base_frame>
+            <robot_base_frame>base_footprint</robot_base_frame>
             <publish_odom>true</publish_odom>
             <publish_odom_tf>true</publish_odom_tf>

File: twowheelbot/designs/lidar.xacro (robot description, xacro)
@@ -4,5 +4,5 @@
   <link name="lidar_link">
     <visual>
-      <origin xyz="0 0 -0.032" rpy="0 0 ${pi}" />
+      <origin xyz="0 0 -0.032" rpy="0 0 0" />
       <geometry>
         <mesh filename="package://twowheelbot/meshes/lidar_link.STL" />
@@ -13,5 +13,5 @@
     </visual>
     <collision>
-      <origin xyz="0 0 -0.032" rpy="0 0 ${pi}" />
+      <origin xyz="0 0 -0.032" rpy="0 0 0" />
       <geometry>
         <mesh filename="package://twowheelbot/meshes/lidar_link.STL" />
@@ -19,5 +19,5 @@
     </collision>
     <inertial>
-      <origin xyz="0 0 -0.032" rpy="0 0 ${pi}" />
+      <origin xyz="0 0 -0.032" rpy="0 0 0" />
       <mass value="0.16538" />
       <inertia ixx="7.519E-05" ixy="-4.8472E-08" ixz="2.886E-08" iyy="7.8865E-05" iyz="-2.1848E-06" izz="0.00010995" />
@@ -57,5 +57,5 @@
         <plugin name = "scan" filename = "libgazebo_ros_ray_sensor.so">
             <ros>
-                <argument>~/out:=scan</argument>
+                <argument>--ros-args --remap ~/out:=scan</argument>
             </ros>
             <output_type>sensor_msgs/LaserScan</output_type>

File: twowheelbot/designs/ros2_control.xacro (robot description, xacro)
@@ -56,6 +56,6 @@
     <gazebo>
         <plugin name="gazebo_ros2_control" filename="libgazebo_ros2_control.so">
-            <parameters>$(find articubot_one)/config/my_controllers.yaml</parameters>
-            <parameters>$(find articubot_one)/config/gaz_ros2_ctl_use_sim.yaml</parameters>
+            <parameters>$(find twowheelbot)/config/my_controllers.yaml</parameters>
+            <parameters>$(find twowheelbot)/config/gaz_ros2_ctl_use_sim.yaml</parameters>
         </plugin>
     </gazebo>

Commit message: ros2 control fixed

File: twowheelbot/designs/amr.urdf.xacro (robot description, xacro)
@@ -1,13 +1,15 @@
 <?xml version="1.0"?>
 <robot xmlns:xacro="http://www.ros.org/wiki/xacro" name="amr_bot">
+    <xacro:arg name="use_ros2_control" default="true"/>
+    <xacro:arg name="sim_mode" default="false"/>
     <xacro:include filename = "amrurdf.urdf" />
+    <xacro:include filename = "lidar.xacro"/>
     <!-- <xacro:include filename = "gz_ctrl.xacro" /> -->
-    <xacro:include filename = "lidar.xacro"/>
     <!-- <xacro:include filename = "imu.xacro"/> -->
-    <!-- <xacro:if value="$(arg use_ros2_control)"> -->
+    <xacro:if value="$(arg use_ros2_control)">
         <xacro:include filename="ros2_control.xacro" />
-    <!-- </xacro:if> -->
-    <!-- <xacro:unless value="$(arg use_ros2_control)">
-        <xacro:include filename="gazebo_control.xacro" />
-    </xacro:unless> -->
+    </xacro:if>
+    <xacro:unless value="$(arg use_ros2_control)">
+        <xacro:include filename="gz_control.xacro" />
+    </xacro:unless>
 </robot>

File: twowheelbot/designs/amrurdf.urdf (robot description, URDF)
Before this commit: robot None, 8 links, 7 joints
Joints:
- joint chassis_joint: origin xyz=0 0 0.045 rpy=0 0 0 -> xyz=0 0 0 rpy=0 0 0
- joint left_wheel_joint: axis 0 0 -1 -> 0 0 1; origin xyz=0 0.234 0.0304999999999985 rpy=-${pi/2} 0 0 -> xyz=0 0.234 0.0304999999999984 rpy=-${pi/2} 0 0
- joint right_wheel_joint: axis 0 0 1 -> 0 0 -1

File: twowheelbot/designs/gz_ctrl.xacro (robot description, xacro)
@@ -6,5 +6,5 @@
             <left_joint>left_wheel_joint</left_joint>
             <right_joint>right_wheel_joint</right_joint>
-            ]<wheel_separation>0.468</wheel_separation>
+            <wheel_separation>0.468</wheel_separation>
             <wheel_diameter>0.07458</wheel_diameter>
             <!-- Limits -->
@@ -13,5 +13,5 @@
             <!-- output -->
             <odometry_frame>odom</odometry_frame>
-            <robot_base_frame>base_link</robot_base_frame>
+            <robot_base_frame>base_footprint</robot_base_frame>
             <publish_odom>true</publish_odom>
             <publish_odom_tf>true</publish_odom_tf>

File: twowheelbot/designs/lidar.xacro (robot description, xacro)
@@ -26,9 +26,10 @@
   <joint name="lidar_link_joint" type="fixed">
     <origin xyz="-0.0063382 0.0016853 0.225" rpy="0 0 1.5164" />
+    <!-- rpy 0 0 -1.5164 -->
     <parent link="base_link" />
     <child link="lidar_link" />
   </joint>
   <gazebo reference="lidar_link">
-    <material>Gazebo/Pink</material>
+    <material>Gazebo/Yellow</material>
     <sensor name="laser" type="ray">
         <pose>0 0 0 0 0 0</pose>
@@ -45,6 +46,6 @@
             </scan>
             <range>
-                <min>0.1</min>
-                <max>11</max>
+                <min>0.3</min>
+                <max>12</max>
                 <!-- <resoluion>0.05</resoluion> -->
             </range>

Commit message: Multi Spawn
Scan topic have been namespaced and they are publishing to slam_toolbox correctly

File: twowheelbot/designs/amr.urdf.xacro (robot description, xacro)
@@ -1,15 +1,9 @@
 <?xml version="1.0"?>
 <robot xmlns:xacro="http://www.ros.org/wiki/xacro" name="amr_bot">
-    <xacro:arg name="use_ros2_control" default="true"/>
+    <xacro:arg name="namespace" default=""/>
     <xacro:arg name="sim_mode" default="false"/>
+    <xacro:property name="namespace" value="$(arg namespace)"/>
     <xacro:include filename = "amrurdf.urdf" />
     <xacro:include filename = "lidar.xacro"/>
-    <!-- <xacro:include filename = "gz_ctrl.xacro" /> -->
-    <!-- <xacro:include filename = "imu.xacro"/> -->
-    <xacro:if value="$(arg use_ros2_control)">
-        <xacro:include filename="ros2_control.xacro" />
-    </xacro:if>
-    <xacro:unless value="$(arg use_ros2_control)">
-        <xacro:include filename="gz_control.xacro" />
-    </xacro:unless>
+    <xacro:include filename = "gz_ctrl.xacro" />
 </robot>

File: twowheelbot/designs/gz_ctrl.xacro (robot description, xacro)
@@ -1,6 +1,11 @@
 <?xml version="1.0"?>
 <robot xmlns:xacro="http://www.ros.org/wiki/xacro">
+    <xacro:arg name="namespace" default=""/>
     <gazebo>
         <plugin name = "diff_drive" filename = "libgazebo_ros_diff_drive.so">
+            <ros>
+                <namespace>${namespace}</namespace>
+                <remapping>/tf:=tf</remapping>
+            </ros>
             <!-- Wheel Info -->
             <left_joint>left_wheel_joint</left_joint>
@@ -9,6 +14,7 @@
             <wheel_diameter>0.07458</wheel_diameter>
             <!-- Limits -->
-            <max_wheel_torque>200</max_wheel_torque>
-            <max_wheel_acceleration>10.0</max_wheel_acceleration>
+            <max_wheel_torque>500</max_wheel_torque>
+            <max_wheel_acceleration>20.0</max_wheel_acceleration>
+            <command_topic>cmd_vel</command_topic>
             <!-- output -->
             <odometry_frame>odom</odometry_frame>

File: twowheelbot/designs/lidar.xacro (robot description, xacro)
@@ -1,5 +1,6 @@
 <?xml version="1.0"?>
 <robot xmlns:xacro="http://www.ros.org/wiki/xacro" >
-    <!-- Lidar Joint -->
+  <xacro:arg name="namespace" default=""/>
+  <!-- Lidar Joint -->
   <link name="lidar_link">
     <visual>
@@ -57,7 +58,9 @@
         </ray>
         <plugin name = "laser_controller" filename = "libgazebo_ros_ray_sensor.so">
-            <ros>
-                <argument>~/out:=scan</argument>
-            </ros>
+          <ros>
+            <namespace>${namespace}</namespace>
+            <!-- <remapping>~/out:=/scan</remapping> -->
+            <remapping>~/out:=scan</remapping>
+          </ros>
             <output_type>sensor_msgs/LaserScan</output_type>
             <frame_name>lidar_link</frame_name>

Commit message: Map Merger Initial Commit
Using the varient package and generated new map merging package

File: twowheelbot/designs/amr.urdf.xacro (robot description, xacro)
@@ -1,9 +1,18 @@
 <?xml version="1.0"?>
-<robot xmlns:xacro="http://www.ros.org/wiki/xacro" name="amr_bot">
-    <xacro:arg name="namespace" default=""/>
+<robot xmlns:xacro="http://www.ros.org/wiki/xacro" name="AME">
+    <xacro:arg name="robot_namespace" default=""/>
     <xacro:arg name="sim_mode" default="false"/>
-    <xacro:property name="namespace" value="$(arg namespace)"/>
+    <!-- <xacro:arg name="use_ros2_control" default = "false"/> -->
+    <!-- Pass namespace as an argument if needed within amrurdf.urdf -->
+    <xacro:property name="robot_namespace" value="$(arg robot_namespace)"/>
     <xacro:include filename = "amrurdf.urdf" />
     <xacro:include filename = "lidar.xacro"/>
     <xacro:include filename = "gz_ctrl.xacro" />
+    <!-- <xacro:include filename = "imu.xacro"/> -->
+    <!-- <xacro:if value="$(arg use_ros2_control)">
+        <xacro:include filename="ros2_control.xacro" />
+    </xacro:if>
+    <xacro:unless value="$(arg use_ros2_control)">
+        <xacro:include filename="gz_ctrl.xacro" />
+    </xacro:unless> -->
 </robot>

File: twowheelbot/designs/gz_ctrl.xacro (robot description, xacro)
@@ -1,9 +1,9 @@
 <?xml version="1.0"?>
 <robot xmlns:xacro="http://www.ros.org/wiki/xacro">
-    <xacro:arg name="namespace" default=""/>
+    <xacro:arg name="robot_namespace" default=""/>
     <gazebo>
         <plugin name = "diff_drive" filename = "libgazebo_ros_diff_drive.so">
             <ros>
-                <namespace>${namespace}</namespace>
+                <namespace>${robot_namespace}</namespace>
                 <remapping>/tf:=tf</remapping>
             </ros>
@@ -14,6 +14,6 @@
             <wheel_diameter>0.07458</wheel_diameter>
             <!-- Limits -->
-            <max_wheel_torque>500</max_wheel_torque>
-            <max_wheel_acceleration>20.0</max_wheel_acceleration>
+            <max_wheel_torque>1200</max_wheel_torque>
+            <max_wheel_acceleration>100.0</max_wheel_acceleration>
             <command_topic>cmd_vel</command_topic>
             <!-- output -->

File: twowheelbot/designs/lidar.xacro (robot description, xacro)
@@ -1,9 +1,9 @@
 <?xml version="1.0"?>
 <robot xmlns:xacro="http://www.ros.org/wiki/xacro" >
-  <xacro:arg name="namespace" default=""/>
+  <xacro:arg name="robot_namespace" default=""/>
   <!-- Lidar Joint -->
   <link name="lidar_link">
     <visual>
-      <origin xyz="0 0 -0.032" rpy="0 0 0" />
+      <origin xyz="0 0 0" rpy="0 0 0" />
       <geometry>
         <mesh filename="package://twowheelbot/meshes/lidar_link.STL" />
@@ -14,5 +14,5 @@
     </visual>
     <collision>
-      <origin xyz="0 0 -0.032" rpy="0 0 0" />
+      <origin xyz="0 0 0" rpy="0 0 0" />
       <geometry>
         <mesh filename="package://twowheelbot/meshes/lidar_link.STL" />
@@ -20,5 +20,5 @@
     </collision>
     <inertial>
-      <origin xyz="0 0 -0.032" rpy="0 0 0" />
+      <origin xyz="0 0 0" rpy="0 0 0" />
       <mass value="0.16538" />
       <inertia ixx="7.519E-05" ixy="-4.8472E-08" ixz="2.886E-08" iyy="7.8865E-05" iyz="-2.1848E-06" izz="0.00010995" />
@@ -26,5 +26,5 @@
   </link>
   <joint name="lidar_link_joint" type="fixed">
-    <origin xyz="-0.0063382 0.0016853 0.225" rpy="0 0 1.5164" />
+    <origin xyz="0.165 0.0016853 0" rpy="0 0 1.5164" />
     <!-- rpy 0 0 -1.5164 -->
     <parent link="base_link" />
@@ -43,5 +43,5 @@
                     <!-- <resolution>0.5</resolution> -->
                     <min_angle>-3.14</min_angle>
-                    <max_angle>3.14</max_angle>
+                    <max_angle>0</max_angle>
                 </horizontal>
             </scan>
@@ -59,5 +59,5 @@
         <plugin name = "laser_controller" filename = "libgazebo_ros_ray_sensor.so">
           <ros>
-            <namespace>${namespace}</namespace>
+            <namespace>${robot_namespace}</namespace>
             <!-- <remapping>~/out:=/scan</remapping> -->
             <remapping>~/out:=scan</remapping>

Commit message: Temporary Push
These changes are subject to revert and new changes

File: twowheelbot/designs/amr.urdf.xacro (robot description, xacro)
@@ -8,11 +8,11 @@
     <xacro:include filename = "amrurdf.urdf" />
     <xacro:include filename = "lidar.xacro"/>
-    <!-- <xacro:include filename = "gz_ctrl.xacro" /> -->
+    <xacro:include filename = "gz_ctrl.xacro" />
     <!-- <xacro:include filename = "imu.xacro"/> -->
-    <xacro:if value="$(arg use_ros2_control)">
+    <!-- <xacro:if value="$(arg use_ros2_control)">
         <xacro:include filename="ros2_control.xacro" />
     </xacro:if>
     <xacro:unless value="$(arg use_ros2_control)">
         <xacro:include filename="gz_ctrl.xacro" />
-    </xacro:unless>
+    </xacro:unless> -->
 </robot>

File: twowheelbot/designs/amrurdf.urdf (robot description, URDF)
Before this commit: robot None, 8 links, 7 joints
Joints:
- joint left_wheel_joint: axis 0 0 1 -> 0 0 -1
- joint lf_caster_joint: axis 0 0 1 -> (none)
- joint lr_caster_joint: axis 0 0 1 -> (none)
- joint rf_caster_joint: axis 0 0 -1 -> (none)
- joint right_wheel_joint: axis 0 0 -1 -> 0 0 1
- joint rr_caster_joint: axis 0 0 -1 -> (none)

File: twowheelbot/designs/gz_ctrl.xacro (robot description, xacro)
@@ -13,5 +13,5 @@
             <right_joint>right_wheel_joint</right_joint>
             <wheel_separation>0.468</wheel_separation>
-            <wheel_diameter>0.07458</wheel_diameter>
+            <wheel_diameter>0.1</wheel_diameter>
             <!-- Limits -->
             <max_wheel_torque>1200</max_wheel_torque>

File: twowheelbot/designs/lidar.xacro (robot description, xacro)
@@ -5,5 +5,5 @@
   <link name="lidar_link">
     <visual>
-      <origin xyz="0 0 0" rpy="0 0 0" />
+      <origin xyz="0 0 -0.025" rpy="0 0 0" />
       <geometry>
         <mesh filename="package://twowheelbot/meshes/lidar_link.STL" />
@@ -14,5 +14,5 @@
     </visual>
     <collision>
-      <origin xyz="0 0 0" rpy="0 0 0" />
+      <origin xyz="0 0 -0.025" rpy="0 0 0" />
       <geometry>
         <mesh filename="package://twowheelbot/meshes/lidar_link.STL" />
@@ -20,5 +20,5 @@
     </collision>
     <inertial>
-      <origin xyz="0 0 0" rpy="0 0 0" />
+      <origin xyz="0 0 -0.025" rpy="0 0 0" />
       <mass value="0.16538" />
       <inertia ixx="7.519E-05" ixy="-4.8472E-08" ixz="2.886E-08" iyy="7.8865E-05" iyz="-2.1848E-06" izz="0.00010995" />
@@ -26,6 +26,5 @@
   </link>
   <joint name="lidar_link_joint" type="fixed">
-    <origin xyz="0.165 0.0016853 0" rpy="0 0 1.5164" />
-    <!-- rpy 0 0 -1.5164 -->
+    <origin xyz="-0.165 0.0016853 0.025" rpy="0 0 -1.5164" />
     <parent link="base_link" />
     <child link="lidar_link" />
@@ -36,5 +35,5 @@
         <pose>0 0 0 0 0 0</pose>
         <visualize>false</visualize>
-        <update_rate>10</update_rate>
+        <update_rate>10.0</update_rate>
         <ray>
             <scan>
@@ -59,6 +58,5 @@
         <plugin name = "laser_controller" filename = "libgazebo_ros_ray_sensor.so">
           <ros>
-            <namespace>${robot_namespace}</namespace>
-            <!-- <remapping>~/out:=/scan</remapping> -->
+            <!-- <namespace>${robot_namespace}</namespace> -->
             <remapping>~/out:=scan</remapping>
           </ros>

Commit message: Map merging Method Update
Better Map merging function than earlier.
A round method, to make the map visible on each of robots

File: twowheelbot/designs/amr.urdf.xacro (robot description, xacro)
@@ -8,11 +8,11 @@
     <xacro:include filename = "amrurdf.urdf" />
     <xacro:include filename = "lidar.xacro"/>
-    <xacro:include filename = "gz_ctrl.xacro" />
+    <!-- <xacro:include filename = "gz_ctrl.xacro" /> -->
     <!-- <xacro:include filename = "imu.xacro"/> -->
-    <!-- <xacro:if value="$(arg use_ros2_control)">
+    <xacro:if value="$(arg use_ros2_control)">
         <xacro:include filename="ros2_control.xacro" />
     </xacro:if>
     <xacro:unless value="$(arg use_ros2_control)">
         <xacro:include filename="gz_ctrl.xacro" />
-    </xacro:unless> -->
+    </xacro:unless>
 </robot>

File: twowheelbot/designs/amrurdf.urdf (robot description, URDF)
Before this commit: robot None, 8 links, 7 joints
Joints:
- removed joint left_wheel_joint
- removed joint right_wheel_joint
- added joint joint_tire_left: type continuous, parent base_link, child left_wheel, origin xyz=0 0.234 0.0304999999999984 rpy=-${pi/2} 0 0, axis 0 0 1
- added joint joint_tire_right: type continuous, parent base_link, child right_wheel, origin xyz=0 -0.234 0.0304999999999984 rpy=${pi/2} 0 0, axis 0 0 -1
- joint lf_caster_joint: axis (none) -> 0 0 1
- joint lr_caster_joint: axis (none) -> 0 0 1
- joint rf_caster_joint: axis (none) -> 0 0 -1
- joint rr_caster_joint: axis (none) -> 0 0 -1

File: twowheelbot/designs/gz_ctrl.xacro (robot description, xacro)
@@ -10,8 +10,8 @@
             </ros>
             <!-- Wheel Info -->
-            <left_joint>left_wheel_joint</left_joint>
-            <right_joint>right_wheel_joint</right_joint>
+            <left_joint>joint_tire_left</left_joint>
+            <right_joint>joint_tire_right</right_joint>
             <wheel_separation>0.468</wheel_separation>
-            <wheel_diameter>0.1</wheel_diameter>
+            <wheel_diameter>0.07458</wheel_diameter>
             <!-- Limits -->
             <max_wheel_torque>1200</max_wheel_torque>

File: twowheelbot/designs/lidar.xacro (robot description, xacro)
@@ -5,5 +5,5 @@
   <link name="lidar_link">
     <visual>
-      <origin xyz="0 0 -0.025" rpy="0 0 0" />
+      <origin xyz="0 0 0" rpy="0 0 0" />
       <geometry>
         <mesh filename="package://twowheelbot/meshes/lidar_link.STL" />
@@ -14,5 +14,5 @@
     </visual>
     <collision>
-      <origin xyz="0 0 -0.025" rpy="0 0 0" />
+      <origin xyz="0 0 0" rpy="0 0 0" />
       <geometry>
         <mesh filename="package://twowheelbot/meshes/lidar_link.STL" />
@@ -20,5 +20,5 @@
     </collision>
     <inertial>
-      <origin xyz="0 0 -0.025" rpy="0 0 0" />
+      <origin xyz="0 0 0" rpy="0 0 0" />
       <mass value="0.16538" />
       <inertia ixx="7.519E-05" ixy="-4.8472E-08" ixz="2.886E-08" iyy="7.8865E-05" iyz="-2.1848E-06" izz="0.00010995" />
@@ -26,5 +26,6 @@
   </link>
   <joint name="lidar_link_joint" type="fixed">
-    <origin xyz="-0.165 0.0016853 0.025" rpy="0 0 -1.5164" />
+    <origin xyz="0.165 0.0016853 0" rpy="0 0 1.5164" />
+    <!-- rpy 0 0 -1.5164 -->
     <parent link="base_link" />
     <child link="lidar_link" />
@@ -33,7 +34,7 @@
     <material>Gazebo/Yellow</material>
     <sensor name="laser" type="ray">
-        <pose>0 0 0 0 0 0</pose>
+        <pose>0 0 0.015 0 0 0</pose>
         <visualize>false</visualize>
-        <update_rate>10.0</update_rate>
+        <update_rate>10</update_rate>
         <ray>
             <scan>
@@ -58,5 +59,6 @@
         <plugin name = "laser_controller" filename = "libgazebo_ros_ray_sensor.so">
           <ros>
-            <!-- <namespace>${robot_namespace}</namespace> -->
+            <namespace>${robot_namespace}</namespace>
+            <!-- <remapping>~/out:=/scan</remapping> -->
             <remapping>~/out:=scan</remapping>
           </ros>
